File: Hardware/Xbee/Xbee.sch (KiCad schematic (older format))
At the start: 44 parts, among them J1 Entrada, J2 Conn_01x05, J3 Pines 1, J4 Pines 2, J5 Programación, J6 Entrada, J7 Salida, K1 DIPxx-1Cxx-51x, Q1 BC338, Q2 BC338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

Commit message: Testing sync
Parts:
- C1, C2: symbol Device:CP1 -> Xbee-rescue:CP1-Device
- D1, D5, D6, D7: symbol Device:LED_ALT -> Xbee-rescue:LED_ALT-Device
- D2, D4: symbol Diode:1N4007 -> Xbee-rescue:1N4007-Diode
- D3: symbol Device:D_Zener_ALT -> Xbee-rescue:D_Zener_ALT-Device
- J1: value Entrada -> Alimentación; symbol Connector:Screw_Terminal_01x02 -> Xbee-rescue:Screw_Terminal_01x02-Connector
- J2: value Conn_01x05 -> Raspberry; symbol Connector_Generic:Conn_01x05 -> Xbee-rescue:Conn_01x05-Connector_Generic
- J3, J4: symbol Connector_Generic:Conn_01x10 -> Xbee-rescue:Conn_01x10-Connector_Generic
- J5: symbol Connector_Generic:Conn_02x05_Counter_Clockwise -> Xbee-rescue:Conn_02x05_Counter_Clockwise-Connector_Generic
- J6, J7: symbol Connector:Screw_Terminal_01x02 -> Xbee-rescue:Screw_Terminal_01x02-Connector
- JP1, JP3: symbol Jumper:Jumper_3_Open -> Xbee-rescue:Jumper_3_Open-Jumper
- JP2, JP4: symbol Jumper:Jumper_2_Open -> Xbee-rescue:Jumper_2_Open-Jumper
- K1: value DIPxx-1Cxx-51x -> Rele12V; symbol Relay:DIPxx-1Cxx-51x -> Xbee-rescue:DIPxx-1Cxx-51x-Relay
- Q1, Q2, Q3: symbol Transistor_BJT:BC338 -> Xbee-rescue:BC338-Transistor_BJT
- R1, R10, R11, R12, R13, R2, R3, R4, R5, R6, R7, R8, R9: symbol Device:R -> Xbee-rescue:R-Device
- RV1, RV2: symbol Device:R_POT -> Xbee-rescue:R_POT-Device
- SW1, SW2: symbol Switch:SW_Push_Dual -> Xbee-rescue:SW_Push_Dual-Switch
- U1: symbol Regulator_Linear:LM317_3PinPackage -> Xbee-rescue:LM317_3PinPackage-Regulator_Linear
- U3: symbol Amplifier_Operational:LM358 -> Xbee-rescue:LM358-Amplifier_Operational

Commit message: Footprint
Parts:
- C1, C2: footprint (none) -> Capacitor_THT:CP_Radial_D5.0mm_P2.50mm
- D1, D5, D6, D7: footprint (none) -> LED_THT:LED_D5.0mm
- D3: footprint (none) -> Diode_THT:D_DO-35_SOD27_P10.16mm_Horizontal
- J1, J6, J7: footprint (none) -> TerminalBlock:TerminalBlock_bornier-2_P5.08mm
- J2: footprint (none) -> Connector_PinHeader_2.54mm:PinHeader_1x05_P2.54mm_Vertical
- J3, J4: footprint (none) -> Connector_PinSocket_2.54mm:PinSocket_1x10_P2.54mm_Vertical
- J5: footprint (none) -> Connector_PinHeader_2.54mm:PinHeader_2x05_P2.54mm_Vertical
- JP1, JP3: footprint (none) -> Connector_PinHeader_2.54mm:PinHeader_1x03_P2.54mm_Vertical
- JP2, JP4: footprint (none) -> Connector_PinHeader_2.54mm:PinHeader_1x02_P2.54mm_Vertical
- K1: footprint Relay_THT:Relay_StandexMeder_DIP_LowProfile -> Relay_THT:Relay_SPDT_SANYOU_SRD_Series_Form_C
- R1, R10, R11, R12, R13, R2, R3, R4, R5, R6, R7, R8, R9: footprint (none) -> Resistor_THT:R_Axial_DIN0207_L6.3mm_D2.5mm_P10.16mm_Horizontal
- RV1, RV2: footprint (none) -> Potentiometer_THT:Potentiometer_Bourns_3386C_Horizontal
- SW1, SW2: footprint (none) -> Button_Switch_THT:SW_TH_Tactile_Omron_B3F-10xx
- U1: footprint (none) -> Package_TO_SOT_THT:TO-220-3_Vertical
- U2: value XBP24CZ7PITB003 -> Xbee; footprint DIP2200W51P200L3294H279Q20P -> XBP24CZ7PITB003:DIP2200W51P200L3294H279Q20P
- U3: footprint (none) -> Package_DIP:DIP-8_W7.62mm_Socket_LongPads
Connections:
- net DSR is gone; now on net DSR-DIO12: J5.2 (Pin_2)
- net DTR is gone; now on net DTR-DIO8: J5.9 (Pin_9)
- net DIO12 renamed DSR-DIO12
- net DIO8 renamed DTR-DIO8
